File: HardWare/Foc.kicad_pcb (KiCad board)
At the start: 4 copper layers, 60 x 45 mm, 147 parts, among them J1 复用Typec, J2 hall, J3 Conn_01x03, J4 hall, J5 Conn_01x03, J6 SWD, J7 inp, J8 XH2.54, J9 SPI_conn, Q1 Q_NMOS_SGD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

Commit message: 改进
Parts:
- removed C49: 2.2uf, Capacitor_SMD:C_0603_1608Metric
- removed R40: 86.6k, Resistor_SMD:R_0603_1608Metric
- added J10: SPI_conn, USER:M1010RS-06P, B.Cu at (90.0, 123.5)
- C20, C24, C25, C26, C27, C28, C29, C7, D3, J1, R15, R16, R20, R23, R25, R50, R51, U1, U7, Y1: moved to F.Cu
- J8: moved to B.Cu
- J9: footprint Connector_Molex:Molex_CLIK-Mate_502386-0670_1x06-1MP_P1.25mm_Horizontal -> USER:M1010RS-06P
- moved D3 74.5 mm to (91.2, 131.4), turned to -90 degrees
- moved R20 70.8 mm to (93.0, 131.5), turned to -90 degrees
- moved J9 65.3 mm to (80.2, 123.5), turned to 0 degrees
- moved J6 55.6 mm to (63.1, 123.3), turned to 90 degrees
- moved J8 47.9 mm to (101.1, 125.0), turned to 180 degrees
- moved J1 44.8 mm to (101.1, 124.4), turned to 180 degrees
- moved U6 33.4 mm to (90.0, 125.6)
- moved D1 32.2 mm to (100.8, 132.3), turned to 180 degrees
- moved U7 31.2 mm to (80.5, 125.6)
- moved C24 28.7 mm to (81.0, 150.1), turned to -90 degrees
- moved R1 25.2 mm to (65.1, 127.7), turned to 90 degrees
- moved Y1 24.6 mm to (83.5, 149.6), turned to 90 degrees
- moved C56 24.4 mm to (86.8, 130.4), turned to -90 degrees
- moved C2 22.9 mm to (57.5, 131.6), turned to 90 degrees
- moved R2 22.7 mm to (67.0, 127.7), turned to -90 degrees
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- renumbered REF** to REFA, REF** to REFB, REF** to REFC, REF** to REFD
Connections:
- U1 pad 55: unconnected-(U1-Pad55) -> /MCU/EXSPI1_CS
Routing:
- net +5V: track 3.70 -> 34.1 mm
- net Net-(Q6-Pad2): track 29.0 -> 2.63 mm, vias 2 -> 0
- net VDC: track 33.1 -> 14.2 mm
- net Net-(D1-Pad1): track 14.5 -> 0.00 mm
- net Net-(Q10-Pad2): track 0.00 -> 13.7 mm
- net Net-(Q8-Pad2): track 0.00 -> 13.3 mm
- net /controller/SN1: track 10.8 -> 23.6 mm, vias 2 -> 4
- net Net-(Q1-Pad2): track 14.6 -> 2.13 mm
- net /motor2/M2_SL_C: track 0.00 -> 9.96 mm, vias 12 -> 14
- net /motor2/M2_SL_B: track 21.9 -> 12.0 mm, vias 14 -> 12
- net Net-(Q4-Pad2): track 22.8 -> 13.8 mm
- net +3.3V: track 0.00 -> 8.48 mm, vias 0 -> 11
- net Net-(C25-Pad1): track 0.00 -> 7.55 mm
- net /motor2/M2_GH_C: track 3.48 -> 10.5 mm, vias 0 -> 2
- net Net-(Q2-Pad2): track 18.5 -> 11.8 mm
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- added copper zone on B.Cu, net GND
- added copper zone on F.Cu, net GND
- added copper zone on In2.Cu, net GND
Other:
- board size 60 x 45 mm -> 60 x 55.2 mm

Commit message: 完成PCB
Parts:
- added G***: LOGO, LOGO, B.Cu at (92.4, 141.4)
- added REF**: ESD-Logo_6.6x6mm_SilkScreen, Symbol:ESD-Logo_6.6x6mm_SilkScreen, F.Cu at (75.0, 131.8)
- added REF**: KiCad-Logo2_8mm_SilkScreen, Symbol:KiCad-Logo2_8mm_SilkScreen, B.Cu at (69.7, 148.5)
- moved C50 27.4 mm to (75.8, 148.2), turned to 0 degrees
- moved C51 25.4 mm to (75.8, 149.7), turned to 0 degrees
- moved C23 25.2 mm to (94.2, 147.9), turned to -90 degrees
- moved C22 25.1 mm to (92.5, 147.9), turned to -90 degrees
- moved C21 25.0 mm to (90.8, 147.9), turned to -90 degrees
- moved C52 23.5 mm to (75.8, 151.2), turned to 0 degrees
- moved D3 18.9 mm to (109.8, 128.5), turned to 0 degrees
- moved R20 17.6 mm to (110.0, 126.7), turned to 0 degrees
- moved R26 1.24 mm to (90.8, 150.9), turned to 90 degrees
- moved R27 1.24 mm to (92.5, 150.9), turned to 90 degrees
- moved R28 1.24 mm to (94.2, 150.9), turned to 90 degrees
Routing:
- net +3.3V: track 8.48 -> 87.4 mm, vias 11 -> 25
- net SPI_SCK: track 1.48 -> 77.7 mm, vias 1 -> 4
- net SPI_MOSI: track 2.91 -> 76.8 mm, vias 1 -> 5
- net GND1: track 0.00 -> 73.2 mm, vias 47 -> 56
- net SPI_MISO: track 2.44 -> 74.2 mm, vias 1 -> 3
- net +3.3VA: track 1.95 -> 70.5 mm, vias 0 -> 3
- net M2_ENC_A: track 0.00 -> 59.4 mm, vias 0 -> 4
- net M1_ENC_A: track 0.00 -> 56.4 mm, vias 0 -> 3
- net M2_ENC_B: track 0.00 -> 54.4 mm, vias 0 -> 4
- net M2_ENC_Z: track 0.00 -> 54.3 mm, vias 0 -> 3
- net M1_ENC_Z: track 0.00 -> 53.6 mm, vias 0 -> 4
- net M1_ENC_B: track 0.00 -> 52.4 mm, vias 0 -> 5
- net EN_GATE: track 1.30 -> 50.2 mm, vias 1 -> 3
- net nFAULT: track 3.32 -> 49.3 mm, vias 1 -> 4
- net GND: track 0.00 -> 45.4 mm, vias 0 -> 11
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- added copper zone on B.Cu, net +3.3V
- added copper zone on In2.Cu, net +3.3V
- removed copper zone on B.Cu, net /controller/SW_BST
- removed copper zone on In2.Cu, net GND
Other:
- board text added: "+3.3"
- board text added: "Brush less"
- board text added: "Clk"
- board text added: "DesignedBy YipingZhu"
- board text added: "Dio"
- board text added: "Gnd"
- board text added: "Powerful!"
- board text added: "Rst"

Commit message: PCB打样
Parts:
- added C156: 100nf, Capacitor_SMD:C_0603_1608Metric, F.Cu at (112.2, 147.5)
- moved G*** 1.63 mm to (91.7, 142.9)
- moved REF** 0.62 mm to (69.1, 148.3)
Routing:
- net +3.3V: track 87.4 -> 88.6 mm, vias 25 -> 32
- net GND: vias 11 -> 47
Other:
- board text added: "FOC-STM32F405 Ver-1.15"
- board text added: "SPI1"
- board text added: "SPI2"
